File: EagleCAD/ReflowMaster.sch (EAGLE design)
At the start: 41 parts, among them Q1 600mA/40V, SW1 SPST_TACT-KMR2, X2 32.768

Commit message: Updated BOM + Schematic pDF + Eagle files with missing part types Changed 12.5pF caps for XTAL to 12pF caps.
Parts:
- added C5: 10nF, microbuilder:CAP_CERAMIC0805-NOOUTLINE
- 13: value BL -> GR
- 2: value BLUE -> YEL
- C2, C4: value 12.5pF -> 12pF
- C3: value 1uF -> 0.1uF
- D1: value (none) -> MBR120
- LDO: value (none) -> AP2112K
- R7: value 2K -> 300R
- R9: value XXX -> 1K2
Connections:
- net T+: now also C5.1
- net T-: now also C5.2
